Commit message: plotting of topology changing objects in box above surface element

File: wall.urdf (robot description, URDF)
Before this commit: robot wall_description, 154 links, 153 joints
Links:
- added link object; collision box size=1.0 1.0 1.0; visual box size=1.0 1.0 1.0
Joints:
- added joint base_to_object: type fixed, parent base_link, child object

Commit message: latest update on body box computation

File: wall.urdf (robot description, URDF)
Before this commit: robot wall_description, 155 links, 154 joints
Links:
- link box10: geometry collision box size=0.170000 0.405009 0.050500; visual box size=0.170000 0.405009 0.050500
- link box100: geometry collision box size=0.225000 0.405009 0.050500; visual box size=0.225000 0.405009 0.050500
- link box101: geometry collision box size=0.150000 0.405009 0.050500; visual box size=0.150000 0.405009 0.050500
- link box102: geometry collision box size=0.225000 0.405009 0.050500; visual box size=0.225000 0.405009 0.050500
- link box103: geometry collision box size=0.225000 0.405009 0.050500; visual box size=0.225000 0.405009 0.050500
- link box104: geometry collision box size=0.225000 0.405009 0.050500; visual box size=0.225000 0.405009 0.050500
- link box105: geometry collision box size=0.225000 0.405009 0.050500; visual box size=0.225000 0.405009 0.050500
- link box106: geometry collision box size=0.225000 0.405009 0.050500; visual box size=0.225000 0.405009 0.050500
- link box107: geometry collision box size=0.130000 0.405009 0.050500; visual box size=0.130000 0.405009 0.050500
- link box108: geometry collision box size=0.170000 0.405009 0.050500; visual box size=0.170000 0.405009 0.050500
- link box109: geometry collision box size=0.170000 0.405009 0.050500; visual box size=0.170000 0.405009 0.050500
- link box11: geometry collision box size=0.170000 0.405009 0.050500; visual box size=0.170000 0.405009 0.050500
- link box110: geometry collision box size=0.225000 0.405009 0.050500; visual box size=0.225000 0.405009 0.050500
- link box111: geometry collision box size=0.150000 0.405009 0.050500; visual box size=0.150000 0.405009 0.050500
- link box112: geometry collision box size=0.225000 0.405009 0.050500; visual box size=0.225000 0.405009 0.050500
- link box113: geometry collision box size=0.150000 0.405009 0.050500; visual box size=0.150000 0.405009 0.050500
- link box114: geometry collision box size=0.130000 0.405009 0.050500; visual box size=0.130000 0.405009 0.050500
- link box115: geometry collision box size=0.170000 0.405009 0.050500; visual box size=0.170000 0.405009 0.050500
- link box116: geometry collision box size=0.200000 0.405009 0.050500; visual box size=0.200000 0.405009 0.050500
- link box117: geometry collision box size=0.190000 0.405009 0.050500; visual box size=0.190000 0.405009 0.050500
- link box118: geometry collision box size=0.225000 0.405009 0.050500; visual box size=0.225000 0.405009 0.050500
- link box119: geometry collision box size=0.225000 0.405009 0.050500; visual box size=0.225000 0.405009 0.050500
- link box12: geometry collision box size=0.225000 0.405009 0.050500; visual box size=0.225000 0.405009 0.050500
- link box120: geometry collision box size=0.180000 0.405009 0.030000; visual box size=0.180000 0.405009 0.030000
- link box121: geometry collision box size=0.225000 0.405009 0.050500; visual box size=0.225000 0.405009 0.050500
- link box122: geometry collision box size=0.225000 0.405009 0.050500; visual box size=0.225000 0.405009 0.050500
- link box123: geometry collision box size=0.225000 0.405009 0.050500; visual box size=0.225000 0.405009 0.050500
- link box124: geometry collision box size=0.225000 0.405009 0.050500; visual box size=0.225000 0.405009 0.050500
- link box125: geometry collision box size=0.225000 0.405009 0.050500; visual box size=0.225000 0.405009 0.050500
- link box126: geometry collision box size=0.225000 0.405009 0.050500; visual box size=0.225000 0.405009 0.050500
- link box127: geometry collision box size=0.225000 0.405009 0.050500; visual box size=0.225000 0.405009 0.050500
- link box128: geometry collision box size=0.170000 0.405009 0.050500; visual box size=0.170000 0.405009 0.050500
- link box129: geometry collision box size=0.170000 0.405009 0.050500; visual box size=0.170000 0.405009 0.050500
- link box13: geometry collision box size=0.170000 0.405009 0.050500; visual box size=0.170000 0.405009 0.050500
- link box130: geometry collision box size=0.170000 0.405009 0.050500; visual box size=0.170000 0.405009 0.050500
- link box131: geometry collision box size=0.225000 0.405009 0.050500; visual box size=0.225000 0.405009 0.050500
- link box132: geometry collision box size=0.225000 0.405009 0.050500; visual box size=0.225000 0.405009 0.050500
- link box133: geometry collision box size=0.225000 0.405009 0.050500; visual box size=0.225000 0.405009 0.050500
- link box134: geometry collision box size=0.225000 0.405009 0.050500; visual box size=0.225000 0.405009 0.050500
- link box135: geometry collision box size=0.225000 0.405009 0.050500; visual box size=0.225000 0.405009 0.050500
- link box136: geometry collision box size=0.225000 0.405009 0.050500; visual box size=0.225000 0.405009 0.050500
- link box137: geometry collision box size=0.225000 0.405009 0.050500; visual box size=0.225000 0.405009 0.050500
- link box138: geometry collision box size=0.225000 0.405009 0.050500; visual box size=0.225000 0.405009 0.050500
- link box139: geometry collision box size=0.225000 0.405009 0.050500; visual box size=0.225000 0.405009 0.050500
- link box14: geometry collision box size=0.200000 0.405009 0.050500; visual box size=0.200000 0.405009 0.050500
- link box140: geometry collision box size=0.225000 0.405009 0.050500; visual box size=0.225000 0.405009 0.050500
- link box141: geometry collision box size=0.170000 0.405009 0.050500; visual box size=0.170000 0.405009 0.050500
- link box142: geometry collision box size=0.170000 0.405009 0.050500; visual box size=0.170000 0.405009 0.050500
- link box143: geometry collision box size=0.170000 0.405009 0.050500; visual box size=0.170000 0.405009 0.050500
- link box144: geometry collision box size=0.170000 0.405009 0.050500; visual box size=0.170000 0.405009 0.050500
- link box145: geometry collision box size=0.170000 0.405009 0.050500; visual box size=0.170000 0.405009 0.050500
- link box15: geometry collision box size=0.200000 0.405009 0.050500; visual box size=0.200000 0.405009 0.050500
- link box16: geometry collision box size=0.225000 0.405009 0.050500; visual box size=0.225000 0.405009 0.050500
- link box17: geometry collision box size=0.225000 0.405009 0.050500; visual box size=0.225000 0.405009 0.050500
- link box18: geometry collision box size=0.225000 0.405009 0.050500; visual box size=0.225000 0.405009 0.050500
- link box19: geometry collision box size=0.225000 0.405009 0.050500; visual box size=0.225000 0.405009 0.050500
- link box20: geometry collision box size=0.225000 0.405009 0.050500; visual box size=0.225000 0.405009 0.050500
- link box21: geometry collision box size=0.225000 0.405009 0.050500; visual box size=0.225000 0.405009 0.050500
- link box22: geometry collision box size=0.225000 0.405009 0.050500; visual box size=0.225000 0.405009 0.050500
- link box23: geometry collision box size=0.225000 0.405009 0.050500; visual box size=0.225000 0.405009 0.050500
- link box24: geometry collision box size=0.150000 0.405009 0.050500; visual box size=0.150000 0.405009 0.050500
- link box25: geometry collision box size=0.225000 0.405009 0.050500; visual box size=0.225000 0.405009 0.050500
- link box26: geometry collision box size=0.170000 0.405009 0.050500; visual box size=0.170000 0.405009 0.050500
- link box27: geometry collision box size=0.225000 0.405009 0.050500; visual box size=0.225000 0.405009 0.050500
- link box28: geometry collision box size=0.225000 0.405009 0.050500; visual box size=0.225000 0.405009 0.050500
- link box29: geometry collision box size=0.225000 0.405009 0.050500; visual box size=0.225000 0.405009 0.050500
- link box3: geometry collision box size=0.225000 0.405009 0.050500; visual box size=0.225000 0.405009 0.050500
- link box30: geometry collision box size=0.225000 0.405009 0.050500; visual box size=0.225000 0.405009 0.050500
- link box31: geometry collision box size=0.150000 0.405009 0.050500; visual box size=0.150000 0.405009 0.050500
- link box32: geometry collision box size=0.225000 0.405009 0.050500; visual box size=0.225000 0.405009 0.050500
- link box33: geometry collision box size=0.225000 0.405009 0.050500; visual box size=0.225000 0.405009 0.050500
- link box34: geometry collision box size=0.150000 0.405009 0.050500; visual box size=0.150000 0.405009 0.050500
- link box35: geometry collision box size=0.170000 0.405009 0.050500; visual box size=0.170000 0.405009 0.050500
- link box36: geometry collision box size=0.225000 0.405009 0.050500; visual box size=0.225000 0.405009 0.050500
- link box37: geometry collision box size=0.225000 0.405009 0.050500; visual box size=0.225000 0.405009 0.050500
- link box38: geometry collision box size=0.225000 0.405009 0.050500; visual box size=0.225000 0.405009 0.050500
- link box39: geometry collision box size=0.225000 0.405009 0.050500; visual box size=0.225000 0.405009 0.050500
- link box4: geometry collision box size=0.225000 0.405009 0.050500; visual box size=0.225000 0.405009 0.050500
- link box40: geometry collision box size=0.225000 0.405009 0.050500; visual box size=0.225000 0.405009 0.050500
- link box41: geometry collision box size=0.225000 0.405009 0.050500; visual box size=0.225000 0.405009 0.050500
- link box42: geometry collision box size=0.170000 0.405009 0.050500; visual box size=0.170000 0.405009 0.050500
- link box43: geometry collision box size=0.170000 0.405009 0.050500; visual box size=0.170000 0.405009 0.050500
- link box44: geometry collision box size=0.180000 0.405009 0.050500; visual box size=0.180000 0.405009 0.050500
- link box45: geometry collision box size=0.170000 0.405009 0.050500; visual box size=0.170000 0.405009 0.050500
- link box46: geometry collision box size=0.225000 0.405009 0.050500; visual box size=0.225000 0.405009 0.050500
- link box47: geometry collision box size=0.225000 0.405009 0.050500; visual box size=0.225000 0.405009 0.050500
- link box48: geometry collision box size=0.225000 0.405009 0.050500; visual box size=0.225000 0.405009 0.050500
- link box49: geometry collision box size=0.225000 0.405009 0.050500; visual box size=0.225000 0.405009 0.050500
- link box5: geometry collision box size=0.150000 0.405009 0.050500; visual box size=0.150000 0.405009 0.050500
- link box50: geometry collision box size=0.225000 0.405009 0.050500; visual box size=0.225000 0.405009 0.050500
- link box51: geometry collision box size=0.190000 0.405009 0.050500; visual box size=0.190000 0.405009 0.050500
- link box52: geometry collision box size=0.190000 0.405009 0.030000; visual box size=0.190000 0.405009 0.030000
- link box53: geometry collision box size=0.225000 0.405009 0.050500; visual box size=0.225000 0.405009 0.050500
- link box54: geometry collision box size=0.225000 0.405009 0.050500; visual box size=0.225000 0.405009 0.050500
- link box55: geometry collision box size=0.225000 0.405009 0.050500; visual box size=0.225000 0.405009 0.050500
- link box56: geometry collision box size=0.225000 0.405009 0.050500; visual box size=0.225000 0.405009 0.050500
- link box57: geometry collision box size=0.225000 0.405009 0.050500; visual box size=0.225000 0.405009 0.050500
- link box58: geometry collision box size=0.225000 0.405009 0.050500; visual box size=0.225000 0.405009 0.050500
- link box59: geometry collision box size=0.130000 0.405009 0.040000; visual box size=0.130000 0.405009 0.040000
- link box6: geometry collision box size=0.120000 0.405009 0.050500; visual box size=0.120000 0.405009 0.050500
- link box60: geometry collision box size=0.190000 0.405009 0.050500; visual box size=0.190000 0.405009 0.050500
- link box61: geometry collision box size=0.225000 0.405009 0.050500; visual box size=0.225000 0.405009 0.050500
- link box62: geometry collision box size=0.225000 0.405009 0.050500; visual box size=0.225000 0.405009 0.050500
- link box63: geometry collision box size=0.225000 0.405009 0.050500; visual box size=0.225000 0.405009 0.050500
- link box64: geometry collision box size=0.225000 0.405009 0.050500; visual box size=0.225000 0.405009 0.050500
- link box65: geometry collision box size=0.170000 0.405009 0.050500; visual box size=0.170000 0.405009 0.050500
- link box66: geometry collision box size=0.160000 0.405009 0.050500; visual box size=0.160000 0.405009 0.050500
- link box67: geometry collision box size=0.160000 0.405009 0.050500; visual box size=0.160000 0.405009 0.050500
- link box68: geometry collision box size=0.225000 0.405009 0.050500; visual box size=0.225000 0.405009 0.050500
- link box69: geometry collision box size=0.225000 0.405009 0.050500; visual box size=0.225000 0.405009 0.050500
- link box7: geometry collision box size=0.120000 0.405009 0.050500; visual box size=0.120000 0.405009 0.050500
- link box70: geometry collision box size=0.225000 0.405009 0.050500; visual box size=0.225000 0.405009 0.050500
- link box71: geometry collision box size=0.225000 0.405009 0.050500; visual box size=0.225000 0.405009 0.050500
- link box72: geometry collision box size=0.225000 0.405009 0.050500; visual box size=0.225000 0.405009 0.050500
- link box73: geometry collision box size=0.225000 0.405009 0.050500; visual box size=0.225000 0.405009 0.050500
- link box74: geometry collision box size=0.225000 0.405009 0.050500; visual box size=0.225000 0.405009 0.050500
- link box75: geometry collision box size=0.225000 0.405009 0.050500; visual box size=0.225000 0.405009 0.050500
- link box76: geometry collision box size=0.190000 0.405009 0.050500; visual box size=0.190000 0.405009 0.050500
- link box77: geometry collision box size=0.190000 0.405009 0.050500; visual box size=0.190000 0.405009 0.050500
- link box78: geometry collision box size=0.225000 0.405009 0.050500; visual box size=0.225000 0.405009 0.050500
- link box79: geometry collision box size=0.225000 0.405009 0.050500; visual box size=0.225000 0.405009 0.050500
- link box8: geometry collision box size=0.150000 0.405009 0.050500; visual box size=0.150000 0.405009 0.050500
- link box80: geometry collision box size=0.170000 0.405009 0.050500; visual box size=0.170000 0.405009 0.050500
- link box81: geometry collision box size=0.130000 0.405009 0.050500; visual box size=0.130000 0.405009 0.050500
- link box82: geometry collision box size=0.225000 0.405009 0.050500; visual box size=0.225000 0.405009 0.050500
- link box83: geometry collision box size=0.225000 0.405009 0.050500; visual box size=0.225000 0.405009 0.050500
- link box84: geometry collision box size=0.225000 0.405009 0.050500; visual box size=0.225000 0.405009 0.050500
- link box85: geometry collision box size=0.225000 0.405009 0.050500; visual box size=0.225000 0.405009 0.050500
- link box86: geometry collision box size=0.225000 0.405009 0.050500; visual box size=0.225000 0.405009 0.050500
- link box87: geometry collision box size=0.170000 0.405009 0.050500; visual box size=0.170000 0.405009 0.050500
- link box88: geometry collision box size=0.170000 0.405009 0.050500; visual box size=0.170000 0.405009 0.050500
- link box89: geometry collision box size=0.225000 0.405009 0.050500; visual box size=0.225000 0.405009 0.050500
- link box9: geometry collision box size=0.130000 0.405009 0.050500; visual box size=0.130000 0.405009 0.050500
- link box90: geometry collision box size=0.225000 0.405009 0.050500; visual box size=0.225000 0.405009 0.050500
- link box91: geometry collision box size=0.225000 0.405009 0.050500; visual box size=0.225000 0.405009 0.050500
- link box92: geometry collision box size=0.225000 0.405009 0.050500; visual box size=0.225000 0.405009 0.050500
- link box93: geometry collision box size=0.225000 0.405009 0.050500; visual box size=0.225000 0.405009 0.050500
- link box94: geometry collision box size=0.225000 0.405009 0.050500; visual box size=0.225000 0.405009 0.050500
- link box95: geometry collision box size=0.225000 0.405009 0.050500; visual box size=0.225000 0.405009 0.050500
- link box96: geometry collision box size=0.225000 0.405009 0.050500; visual box size=0.225000 0.405009 0.050500
- link box97: geometry collision box size=0.170000 0.405009 0.050500; visual box size=0.170000 0.405009 0.050500
- link box98: geometry collision box size=0.170000 0.405009 0.050500; visual box size=0.170000 0.405009 0.050500
- link box99: geometry collision box size=0.225000 0.405009 0.050500; visual box size=0.225000 0.405009 0.050500

Commit message: layered boxes implemented, verified with wall environment

File: wall.urdf (robot description, URDF)
Before this commit: robot wall_description, 155 links, 154 joints
Links:
- removed link object
Joints:
- removed joint base_to_object

Commit message: add connector module for path optimization

File: wall.urdf (robot description, URDF)
Before this commit: robot wall_description, 154 links, 153 joints
Links:
- removed link wall_floor2
- link wall_floor1: geometry collision box size=2.0 6.0 0.1; visual box size=2.0 6.0 0.1
Joints:
- removed joint base_to_wall_floor2
